File: BreadboardPwr/Schematics/BreadboardPwr.sch (KiCad schematic (older format))
At the start: 16 parts, among them J1 Serial, J2 Power, J3 USB_B_Micro, SW1 SW_DIP_x01, U1 otter_CH330, U2 HX4056, U3 TLV1117-33

Commit message: Updated Min dev
Parts:
- removed SW1: SW_DIP_x01, Buttons_Switches_SMD:SK-3296S_switch, symbol Switch:SW_DIP_x01
- added D1, D2, D3, D4: LED, LED_SMD:LED_0603_1608Metric, symbol Device:LED
- added J4: Left, Connector_PinHeader_2.54mm:PinHeader_2x03_P2.54mm_Vertical, symbol Connector_Generic:Conn_02x03_Odd_Even
- added J5: Right, Connector_PinHeader_2.54mm:PinHeader_2x03_P2.54mm_Vertical, symbol Connector_Generic:Conn_02x03_Odd_Even
- added RN1: R_Pack04, Resistor_SMD:R_Array_Convex_4x0603, symbol Device:R_Pack04
- added SW1: SW_DPDT_x2, BreadBoardPwr:SK-3296S_switch, symbol Switch:SW_DPDT_x2
- BT1: footprint Battery_Holders:Keystone_3009_1x2450-CoinCell -> Battery:BatteryHolder_Keystone_3008_1x2450; symbol badge-rescue:Battery_Cell -> BreadboardPwr-rescue:Battery_Cell-badge-rescue
- C1, C2, C3, C4, C5, C6: footprint Capacitors_SMD:C_0805_HandSoldering -> Capacitor_SMD:C_0805_2012Metric; symbol badge-rescue:C -> BreadboardPwr-rescue:C-badge-rescue
- J1, J2: footprint Wire_Pads:SolderWirePad_2x_1mmDrill -> Connector_PinHeader_2.54mm:PinHeader_1x02_P2.54mm_Vertical; symbol badge-rescue:Conn_01x02 -> BreadboardPwr-rescue:Conn_01x02-badge-rescue
- J3: footprint Connectors_USB:USB_Micro-B_Jing -> CH552:USB_Micro-B_Jing
- R1: footprint Resistors_SMD:R_0805 -> Resistor_SMD:R_0805_2012Metric
- R2: footprint Resistors_SMD:R_0805_HandSoldering -> Resistor_SMD:R_0805_2012Metric; symbol badge-rescue:R -> BreadboardPwr-rescue:R-badge-rescue
- U1: footprint Housings_SOIC:SOIC-8-1EP_3.9x4.9mm_Pitch1.27mm -> Package_SO:SOIC-8_3.9x4.9mm_P1.27mm; symbol badge-rescue:otter_CH330-CH330-cache -> BreadboardPwr-rescue:otter_CH330-CH330-cache-badge-rescue
- U2: footprint Badge:HX4056 -> Package_SO:SOIC-8-1EP_3.9x4.9mm_P1.27mm_EP2.29x3mm; symbol badge-rescue:HX4056 -> BreadboardPwr-rescue:HX4056-badge-rescue
- U3: footprint TO_SOT_Packages_SMD:SOT-223-3_TabPin2 -> Package_TO_SOT_SMD:SOT-223-3_TabPin2
Connections:
- net PwrIn: now also SW1.2 (B)
- net VBUS: now also RN1.5 (R4.2), RN1.6 (R3.2), SW1.1 (A)
- net VDD: now also J4.2 (Pin_2), J4.4 (Pin_4), J4.6 (Pin_6), J5.2 (Pin_2), J5.4 (Pin_4), J5.6 (Pin_6), RN1.7 (R2.2), RN1.8 (R1.2)
- net VSS: now also D3.1 (K), D4.1 (K), J4.1 (Pin_1), J4.3 (Pin_3), J4.5 (Pin_5), J5.1 (Pin_1), J5.3 (Pin_3), J5.5 (Pin_5)
- net Stat1: now reaches U2.7 (STAT1)
- net Stat1: now also D1.1 (K)
- net IO27 renamed Stat2
- net Stat2: now also D2.1 (K)
- new net: D1.2 (A), RN1.4 (R4.1)
- new net: D2.2 (A), RN1.3 (R3.1)
- new net: D3.2 (A), RN1.2 (R2.1)
- new net: D4.2 (A), RN1.1 (R1.1)
- no-connect marks 3 -> 4
Other:
- moved on the sheet: J1, J2
