File: Tests/STM32F030Minimal/STM32F030Minimal.sch (KiCad schematic (older format))
At the start: 14 parts, among them J1 Aux, J2 Left, J3 Right, J4 Prog, SW1 SW_DIP_x01, U1 STM32F030F4Px, Y1 8MHz

Commit message: Updated Min dev
Parts:
- C1, C2: value C_Small -> 20pF
Changed lines of the file:
@@
 EESchema Schematic File Version 4
+LIBS:STM32F030Minimal-cache
 EELAYER 29 0
 EELAYER END
@@
 P 5050 3550
 F 0 "C1" V 4821 3550 50  0000 C CNN
-F 1 "C_Small" V 4912 3550 50  0000 C CNN
+F 1 "20pF" V 4912 3550 50  0000 C CNN
 F 2 "Capacitor_SMD:C_0805_2012Metric" H 5050 3550 50  0001 C CNN
 F 3 "~" H 5050 3550 50  0001 C CNN
@@
 P 5050 3750
 F 0 "C2" V 4821 3750 50  0000 C CNN
-F 1 "C_Small" V 4912 3750 50  0000 C CNN
+F 1 "20pF" V 4912 3750 50  0000 C CNN
 F 2 "Capacitor_SMD:C_0805_2012Metric" H 5050 3750 50  0001 C CNN
 F 3 "~" H 5050 3750 50  0001 C CNN
