File: Tests/STM32F411Minimal/STM32F411Minimal.sch (KiCad schematic (older format))
At the start: 33 parts, among them J1 One, J2 Two, J3 Three, J4 Four, J5 Prog, J6 BreadboardPwr, SW1 SW_DIP_x01, U1 STM32F411RETx, Y1 Crystal_GND24, Y2 32.768kHz

Commit message: Recieved V1
Parts:
- Y1: value Crystal_GND24 -> 8MHz
Changed lines of the file:
@@
 U 1 1 5D02EA76
 P 6350 3150
-F 0 "Y1" V 6304 3394 50  0000 L CNN
-F 1 "Crystal_GND24" V 6395 3394 50  0000 L CNN
+F 0 "Y1" V 6650 2950 50  0000 L CNN
+F 1 "8MHz" V 6550 2950 50  0000 L CNN
 F 2 "Crystal:Crystal_SMD_SeikoEpson_TSX3225-4Pin_3.2x2.5mm" H 6350 3150 50  0001 C CNN
 F 3 "~" H 6350 3150 50  0001 C CNN
@@
 P 6550 3150
 F 0 "#PWR019" H 6550 3000 50  0001 C CNN
-F 1 "VSS" V 6567 3278 50  0000 L CNN
+F 1 "VSS" V 6500 3300 50  0000 L CNN
 F 2 "" H 6550 3150 50  0001 C CNN
 F 3 "" H 6550 3150 50  0001 C CNN
