File: Tests/LN4890-AmpD/LN4890.sch (KiCad schematic (older format))
At the start: 31 parts

Commit message: Moving between computers, many changes
Parts:
- removed C? (x2): 1uF, Capacitor_SMD:C_0805_2012Metric, symbol badge-rescue:C
- removed C? (x5): 100nF, Capacitor_SMD:C_0805_2012Metric, symbol Device:C_Small
- removed C?: 10uF, Capacitor_SMD:C_0805_2012Metric, symbol Device:C_Small
- removed C?: 1uF, Capacitor_SMD:C_0805_2012Metric, symbol Device:C_Small
- removed J?: USB_B_Micro, CH552:USB_Micro-B_Jing, symbol Connector:USB_B_Micro
- removed J?: Expansion, Connector_PinHeader_2.54mm:PinHeader_1x05_P2.54mm_Vertical, symbol badge-rescue:Conn_01x05
- removed J?: i2c, Connector_PinHeader_2.54mm:PinHeader_1x03_P2.54mm_Vertical, symbol Connector_Generic:Conn_01x03
- removed J?: Prog, Connector_PinHeader_2.54mm:PinHeader_1x04_P2.54mm_Vertical, symbol badge-rescue:Conn_01x04
- removed J?: Conn_01x03, Connector_PinHeader_2.54mm:PinHeader_1x03_P2.54mm_Vertical, symbol Connector_Generic:Conn_01x03
- removed J?: Conn_01x02, symbol badge-rescue:Conn_01x02
- removed L?: Bead, symbol Device:L
- removed LS?: Speaker, symbol Device:Speaker
- removed R?: 10k, Resistor_SMD:R_0805_2012Metric, symbol Device:R_Small
- removed R? (x2): 2k, Resistor_SMD:R_0805_2012Metric, symbol Device:R_Small
- removed SW?: SW_SPDT, BreadBoardPwr:SK-3296S_switch, symbol Switch:SW_SPDT
- removed U?: TLV1117-33, Package_TO_SOT_SMD:SOT-223-3_TabPin2, symbol Regulator_Linear:TLV1117-33
- removed U?: STM32L052C8Tx, Package_QFP:LQFP-48_7x7mm_P0.5mm, symbol MCU_ST_STM32L0:STM32L052C8Tx
- added J1: Out, TerminalBlock:TerminalBlock_Altech_AK300-2_P5.00mm, symbol badge-rescue:Conn_01x02
- added J3: Conn_01x04, Connector_PinHeader_2.54mm:PinHeader_1x04_P2.54mm_Vertical, symbol badge-rescue:Conn_01x04
- C1, C2, C3: renamed from C?; footprint (none) -> Capacitor_SMD:C_0805_2012Metric
- J2: renamed from J?; footprint (none) -> Connector_PinHeader_2.54mm:PinHeader_1x01_P2.54mm_Vertical
- R1, R2, R3: renamed from R?; footprint (none) -> Resistor_SMD:R_0805_2012Metric
- U1: renamed from U?; footprint (none) -> Package_SO:TSSOP-8_3x3mm_P0.65mm
Connections:
- net Audio: now also J3.1 (Pin_1)
- net Shutdown: now also J3.2 (Pin_2)
- net VCC: now also J3.4 (Pin_4)
- net VSS: now also J3.3 (Pin_3)
- net at R3.1, U1.5 (VO1): now also J1.2 (Pin_2)
- net at U1.8 (VO2): now also J1.1 (Pin_1)
- no-connect marks 26 -> 0
