File: SAO/ZeldaStones/GoronRuby/Schematics/Goron's_Ruby.kicad_pcb (KiCad board)
At the start: 2 copper layers, 37.5 x 36.6 mm, 11 parts, among them J1 Conn_02x03_Odd_Even

Commit message: Making stencils
Parts:
- removed the G*** at (147.2, 107.8) (x4)
- added G*** (x4): LOGO, LOGO, F.Cu at (147.2, 107.8)
Changed lines of the file:
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@@
     (visible_elements FFFFFF7F)
     (pcbplotparams
-      (layerselection 0x010f0_ffffffff)
+      (layerselection 0x010f4_ffffffff)
       (usegerberextensions false)
       (usegerberattributes false)
