File: SAO/ZeldaStones/ZoraSaphire/Schematics/ZoraSapphire.kicad_pcb (KiCad board)
At the start: 2 copper layers, 39.6 x 34.9 mm, 11 parts, among them J1 Conn_02x03_Odd_Even

Commit message: Making stencils
Parts:
- removed the G*** at (151.6, 96.7) (x4)
- added G*** (x4): LOGO, LOGO, F.Cu at (151.6, 96.7)
Changed lines of the file:
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@@
     (visible_elements FFFFFF7F)
     (pcbplotparams
-      (layerselection 0x010f0_ffffffff)
+      (layerselection 0x010f4_ffffffff)
       (usegerberextensions false)
       (usegerberattributes false)
