File: WordClock/Schematics/Top/WordClock.kicad_pcb (KiCad board)
At the start: 2 copper layers, 98.5 x 98.4 mm, 5 parts

Commit message: Updates, added schematic pdf
Parts:
- removed the G*** at (141.9, 101.0) (x4)
- added G*** (x4): LOGO, LOGO, F.Cu at (141.9, 101.0)
- added J1: Conn_01x01, TestPoint:TestPoint_Pad_1.0x1.0mm, B.Cu at (109.6, 146.9)
- added J2: Conn_01x01, TestPoint:TestPoint_Pad_1.0x1.0mm, B.Cu at (109.6, 75.5)
- added J3: Conn_02x03_Odd_Even, Connector_PinSocket_2.54mm:PinSocket_2x03_P2.54mm_Vertical, F.Cu at (101.5, 56.9)
- added J4: Conn_02x03_Odd_Even, Connector_PinSocket_2.54mm:PinSocket_2x03_P2.54mm_Vertical, F.Cu at (128.7, 56.9)
- added J5: Conn_02x03_Odd_Even, Connector_PinSocket_2.54mm:PinSocket_2x03_P2.54mm_Vertical, F.Cu at (156.0, 56.9)
- added J6: Conn_02x03_Odd_Even, Connector_PinSocket_2.54mm:PinSocket_2x03_P2.54mm_Vertical, F.Cu at (183.3, 56.9)
- added J7: Conn_01x01, TestPoint:TestPoint_Pad_1.0x1.0mm, B.Cu at (175.9, 146.9)
- added J8: Conn_01x01, TestPoint:TestPoint_Pad_1.0x1.0mm, B.Cu at (175.9, 75.5)
Routing:
- net +3V3: track 0.00 -> 209.3 mm
- net GND: track 0.00 -> 195.1 mm
Other:
- board text added: "1"
