File: WordClock/Schematics/Bottom/WordClockBottom.kicad_pcb (KiCad board)
At the start: 2 copper layers, 98.5 x 89.5 mm, 6 parts

Commit message: Progress on Dragos badge
Parts:
- removed the G*** at (0.00, 0.00) (x6)
- added <- Power: Power, BreadBoardPwr:SK-3296S_switch, B.Cu at (93.7, 79.5)
- added C1: 4.7uF, Capacitor_SMD:C_0805_2012Metric, B.Cu at (142.5, 116.8)
- added C2: 1uF, Capacitor_SMD:C_0805_2012Metric, B.Cu at (160.1, 112.5)
- added C3: 100nF, Capacitor_SMD:C_0805_2012Metric, B.Cu at (142.5, 113.6)
- added C4: 10nF, Capacitor_SMD:C_0805_2012Metric, B.Cu at (160.1, 116.0)
- added C5: 100nF, Capacitor_SMD:C_0805_2012Metric, B.Cu at (152.5, 108.0)
- added C6: 20pF, Capacitor_SMD:C_0805_2012Metric, B.Cu at (156.0, 102.0)
- added C7: 20pF, Capacitor_SMD:C_0805_2012Metric, B.Cu at (161.1, 102.0)
- added C8: 1uF, Capacitor_SMD:C_0805_2012Metric, B.Cu at (125.6, 137.0)
- added C9: 1uF, Capacitor_SMD:C_0805_2012Metric, B.Cu at (130.1, 137.0)
- added G*** (x3): LOGO, LOGO, F.Cu at (0.00, 0.00)
- added G*** (x3): LOGO, LOGO, F.Cu at (140.2, 90.9)
- added Hour: Hour, Button_Switch_SMD:SW_Push_1P1T_NO_CK_KSC6xxJ, B.Cu at (181.6, 111.6)
- added J1: Prog, Connector_PinHeader_2.54mm:PinHeader_1x04_P2.54mm_Vertical, B.Cu at (95.0, 112.0)
- added J2: Conn_01x02, Connector_PinHeader_2.54mm:PinHeader_1x02_P2.54mm_Vertical, B.Cu at (119.0, 137.0)
- added J3: USB_C_Receptacle, Tests:USB_C_Receptical-Jing, B.Cu at (139.2, 135.8)
- added J5: Left, Connector_PinHeader_2.54mm:PinHeader_1x05_P2.54mm_Vertical, B.Cu at (187.8, 96.1)
- added LED1: WS2812B, BsidesIowa:WS2812B-Sunken, B.Cu at (115.3, 71.0)
- added LED10: WS2812B, BsidesIowa:WS2812B-Sunken, B.Cu at (136.5, 97.3)
- added LED11: WS2812B, BsidesIowa:WS2812B-Sunken, B.Cu at (168.5, 97.3)
- added LED12: WS2812B, BsidesIowa:WS2812B-Sunken, B.Cu at (114.0, 105.7)
- added LED13: WS2812B, BsidesIowa:WS2812B-Sunken, B.Cu at (140.2, 105.7)
- added LED14: WS2812B, BsidesIowa:WS2812B-Sunken, B.Cu at (168.3, 105.7)
- added LED15: WS2812B, BsidesIowa:WS2812B-Sunken, B.Cu at (106.4, 114.2)
- added LED16: WS2812B, BsidesIowa:WS2812B-Sunken, B.Cu at (133.4, 114.2)
- added LED17: WS2812B, BsidesIowa:WS2812B-Sunken, B.Cu at (168.5, 114.2)
- added LED18: WS2812B, BsidesIowa:WS2812B-Sunken, B.Cu at (109.1, 122.5)
- added LED19: WS2812B, BsidesIowa:WS2812B-Sunken, B.Cu at (133.8, 122.5)
- added LED2: WS2812B, BsidesIowa:WS2812B-Sunken, B.Cu at (142.8, 71.0)
- added LED20: WS2812B, BsidesIowa:WS2812B-Sunken, B.Cu at (165.3, 122.5)
- added LED21: WS2812B, BsidesIowa:WS2812B-Sunken, B.Cu at (118.1, 130.6)
- added LED22: WS2812B, BsidesIowa:WS2812B-Sunken, B.Cu at (162.9, 130.7)
- added LED3: WS2812B, BsidesIowa:WS2812B-Sunken, B.Cu at (167.8, 71.0)
- added LED4: WS2812B, BsidesIowa:WS2812B-Sunken, B.Cu at (119.6, 79.4)
- added LED5: WS2812B, BsidesIowa:WS2812B-Sunken, B.Cu at (164.7, 79.4)
- added LED6: WS2812B, BsidesIowa:WS2812B-Sunken, B.Cu at (105.6, 88.8)
- added LED7: WS2812B, BsidesIowa:WS2812B-Sunken, B.Cu at (141.2, 88.8)
- added LED8: WS2812B, BsidesIowa:WS2812B-Sunken, B.Cu at (177.7, 88.8)
- added LED9: WS2812B, BsidesIowa:WS2812B-Sunken, B.Cu at (109.6, 97.3)
- added Prog: Prog, BreadBoardPwr:SK-3296S_switch, B.Cu at (93.6, 96.6)
- added Quarter: Quarter, Button_Switch_SMD:SW_Push_1P1T_NO_CK_KSC6xxJ, B.Cu at (181.7, 101.6)
- added R1: 10k, Resistor_SMD:R_0805_2012Metric, B.Cu at (148.4, 131.0)
- added R2: 10k, Resistor_SMD:R_0805_2012Metric, B.Cu at (101.6, 95.5)
- added R3: 10k, Resistor_SMD:R_0805_2012Metric, B.Cu at (148.5, 134.4)
- added REF**: SolderWirePad_1x01_Drill2.5mm, Connector_Wire:SolderWirePad_1x01_Drill2.5mm, F.Cu at (141.0, 56.0)
- added REF**: TestPoint_Pad_1.0x1.0mm, TestPoint:TestPoint_Pad_1.0x1.0mm, F.Cu at (107.8, 65.4)
- added REF**: TestPoint_Pad_1.0x1.0mm, TestPoint:TestPoint_Pad_1.0x1.0mm, F.Cu at (107.8, 136.8)
- added REF**: TestPoint_Pad_1.0x1.0mm, TestPoint:TestPoint_Pad_1.0x1.0mm, F.Cu at (174.2, 136.8)
- added REF**: TestPoint_Pad_1.0x1.0mm, TestPoint:TestPoint_Pad_1.0x1.0mm, F.Cu at (174.2, 65.4)
- added Reset: Reset, Button_Switch_SMD:SW_Push_1P1T_NO_CK_KSC6xxJ, B.Cu at (181.6, 121.5)
- added U1: STM32F042F6Px, Package_SO:TSSOP-20_4.4x6.5mm_P0.65mm, B.Cu at (151.5, 115.2)
- added U2: TLV1117-33, Package_TO_SOT_SMD:SOT-223-3_TabPin2, B.Cu at (128.0, 130.2)
- added Y1: 8MHz, Crystal:Crystal_SMD_5032-2Pin_5.0x3.2mm, B.Cu at (158.7, 107.5)
Routing:
- net PA0: track 0.00 -> 157.4 mm, vias 0 -> 1
- net VSS: track 0.00 -> 138.3 mm, vias 0 -> 18
- net RST: track 0.00 -> 112.5 mm, vias 0 -> 1
- net VCC: track 0.00 -> 108.1 mm, vias 0 -> 26
- net Net-(C9-Pad1): track 0.00 -> 95.3 mm, vias 0 -> 4
- net Net-(LED3-Pad2): track 0.00 -> 83.2 mm
- net Net-(LED21-Pad2): track 0.00 -> 67.3 mm, vias 0 -> 2
- net BOOT0: track 0.00 -> 66.5 mm
- net Net-(LED8-Pad2): track 0.00 -> 64.6 mm, vias 0 -> 2
- net Net-(LED4-Pad2): track 0.00 -> 63.2 mm
- net PA1: track 0.00 -> 61.9 mm, vias 0 -> 1
- net Net-(LED17-Pad2): track 0.00 -> 60.4 mm, vias 0 -> 2
- net Net-(LED14-Pad2): track 0.00 -> 58.6 mm, vias 0 -> 2
- net Net-(LED7-Pad2): track 0.00 -> 58.5 mm
- net SWDIO: track 0.00 -> 57.4 mm
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- added copper zone on F.Cu, net VCC
- added copper zone on B.Cu, net VSS
