File: WordClock/Schematics/Bottom/WordClockBottom.sch (KiCad schematic (older format))
At the start: 46 parts

Commit message: Progress on Dragos badge
Parts:
- removed SW?: SW_DIP_x01, Button_Switch_SMD:SW_Push_1P1T_NO_CK_KSC7xxJ, symbol Switch:SW_DIP_x01
- added SW1: Hour, Button_Switch_SMD:SW_Push_1P1T_NO_CK_KSC6xxJ, symbol Switch:SW_Push
- added SW4: Quarter, Button_Switch_SMD:SW_Push_1P1T_NO_CK_KSC6xxJ, symbol Switch:SW_Push
- added SW5: Reset, Button_Switch_SMD:SW_Push_1P1T_NO_CK_KSC6xxJ, symbol Switch:SW_Push
- LED1, LED10, LED11, LED12, LED13, LED14, LED15, LED16, LED17, LED18, LED19, LED2, LED20, LED21, LED22, LED3, LED4, LED5, LED6, LED7, LED8, LED9: renamed from LED?; footprint LEDs:LED_WS2812B-PLCC4 -> BsidesIowa:WS2812B-Sunken
- gave numbers to parts that had none: 23
Connections:
- net VDDA is gone; now on net +5V: C8.1, U2.3 (VI)
- net PA0: now also LED1.4 (DIN)
- net PA6: now also SW1.1
- net PA7: now also SW4.1
- net RST: now also SW5.1
- net VSS: now also SW1.2, SW4.2, SW5.2
- no-connect marks 11 -> 12
Other:
- moved on the sheet: C1, C2, C3, C4, C5, C6, C7, C8, C9, J1, J2, J3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
