File: Badges/Dragos/Schematics/V1-Deprecated/dragos.sch (KiCad schematic (older format))
At the start: 59 parts, among them J1 One, J2 Two, J3 CC2530-ISP, J4 Three, J5 Prog, J7 USB_C_Receptacle, J8 Four, J9 BreadboardPwr, SW1 SW_DIP_x01, SW2 SW_DIP_x01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

Commit message: D Badge V2 ordered
Parts:
- BT1: symbol badge-rescue:Battery_Cell -> dragos-rescue:Battery_Cell-badge-rescue
- C10, C11, C8, C9: symbol badge-rescue:C -> dragos-rescue:C-badge-rescue
- R6: symbol badge-rescue:R -> dragos-rescue:R-badge-rescue
- U3: symbol badge-rescue:HX4056 -> dragos-rescue:HX4056-badge-rescue
Changed lines of the file:
@@
 LIBS:74xx
 LIBS:dragos-cache
-EELAYER 29 0
+EELAYER 30 0
 EELAYER END
 $Descr A3 16535 11693
@@
 	2550 3500 2850 3500
 $Comp
-L badge-rescue:Battery_Cell BT1
+L dragos-rescue:Battery_Cell-badge-rescue BT1
 U 1 1 5AD687D0
 P 6900 10550
@@
 	7900 10400 7800 10400
 $Comp
-L badge-rescue:C C10
+L dragos-rescue:C-badge-rescue C10
 U 1 1 5C332E52
 P 7800 10550
@@
 	7800 10400 7700 10400
 $Comp
-L badge-rescue:C C11
+L dragos-rescue:C-badge-rescue C11
 U 1 1 5C332F0A
 P 8600 10550
@@
 $EndComp
 $Comp
-L badge-rescue:C C9
+L dragos-rescue:C-badge-rescue C9
 U 1 1 5C33B6A8
 P 6000 10250
@@
 	5800 10400 6000 10400
 $Comp
-L badge-rescue:C C8
+L dragos-rescue:C-badge-rescue C8
 U 1 1 5C344660
 P 4600 10250
@@
 $EndComp
 $Comp
-L badge-rescue:R R6
+L dragos-rescue:R-badge-rescue R6
 U 1 1 5C37B5B5
 P 5950 10500
@@
 NoConn ~ 3450 3200
 $Comp
-L badge-rescue:HX4056 U3
+L dragos-rescue:HX4056-badge-rescue U3
 U 1 1 5C6DE973
 P 5400 10500
