File: Badges/Dragos/Schematics/V2/dragos.kicad_pcb (KiCad board)
At the start: 2 copper layers, 130.4 x 110.8 mm, 28 parts, among them J2 Oled, J3 AA Batteries, J4 Conn_02x04_Odd_Even, J7 USB_C_Receptacle, J9 BreadboardPwr, SW2 SW_DIP_x01, SW4 SW_DIP_x01, U1 BMD-340-A-R, U2 TLV1117-33, U5 K1-5202UA-03(5Way_Switch)

Commit message: Firmware in progress
Parts:
- removed the G*** at (0.00, 0.00) (x2)
- removed J3: AA Batteries, Dragos:AA
- added G*** (x2): LOGO, LOGO, F.Cu at (0.00, 0.00)
- added J1: Conn_01x02, Connector_PinHeader_2.54mm:PinHeader_1x02_P2.54mm_Vertical, F.Cu at (134.2, 100.3)
- added Ref**: Val**, NFCBuisness:W, B.Cu at (163.6, 139.8)
Connections:
- U1 pad 66: VCC -> +5V
Routing:
- net +5V: track 27.0 -> 112.5 mm, vias 0 -> 2
- net Net-(J3-Pad2): track 38.1 -> 0.00 mm
- net Net-(D1-Pad3): track 111.8 -> 109.3 mm
- net SCL: track 84.1 -> 81.8 mm
- net Left: track 55.4 -> 53.3 mm, vias 2 -> 1
- net VCC: track 270.2 -> 268.6 mm, vias 3 -> 5
- net SDA: track 83.8 -> 82.3 mm
- net D-: track 95.2 -> 93.8 mm
- net D+: track 95.9 -> 94.5 mm
- net VDD: track 92.8 -> 94.0 mm
- net Eye: track 107.1 -> 106.0 mm
- net Down: track 59.5 -> 58.5 mm
- net Net-(D1-Pad2): track 104.9 -> 105.5 mm
- net P1.04: track 16.3 -> 16.0 mm, vias 0 -> 2
Other:
- board text added: "- +"
- board text added: "JLCJLCJLCJLC"
- board text added: "RMA Electronics 2019"
