File: Badges/Dragos/Schematics/V2/dragos.sch (KiCad schematic (older format))
At the start: 21 parts, among them J2 Oled, J3 AA Batteries, J4 Conn_02x04_Odd_Even, J7 USB_C_Receptacle, J9 BreadboardPwr, SW2 SW_DIP_x01, SW4 SW_DIP_x01, U1 BMD-340-A-R, U2 TLV1117-33, U5 K1-5202UA-03(5Way_Switch)

Commit message: Firmware in progress
Parts:
- removed J3: AA Batteries, Dragos:AA, symbol badge-rescue:Conn_01x04
- added J1: Conn_01x02, symbol badge-rescue:Conn_01x02
- R14: value 4k7 -> 1k
Connections:
- net +5V: now also U1.66 (VBUS)
- net VCC: no longer U1.66 (VBUS)
- net VDD: now also J1.2 (Pin_2)
- net VSS: now also J1.1 (Pin_1)
Changed lines of the file:
@@
 LIBS:74xx
 LIBS:dragos-cache
-EELAYER 29 0
+EELAYER 30 0
 EELAYER END
 $Descr A3 16535 11693
@@
 P 6500 4750
 F 0 "R14" V 6304 4750 50  0000 C CNN
-F 1 "4k7" V 6395 4750 50  0000 C CNN
+F 1 "1k" V 6395 4750 50  0000 C CNN
 F 2 "Resistor_SMD:R_0805_2012Metric" H 6500 4750 50  0001 C CNN
 F 3 "~" H 6500 4750 50  0001 C CNN
@@
 Text GLabel 6100 5600 0    50   Input ~ 0
 Down
-Text GLabel 6100 5700 0    50   Input ~ 0
-Up
 Text GLabel 6100 5900 0    50   Input ~ 0
 Right
@@
 	4400 8800 4500 8800
 $Comp
-L power:VSS #PWR010
-U 1 1 5DA16F1E
-P 3250 8000
-F 0 "#PWR010" H 3250 7850 50  0001 C CNN
-F 1 "VSS" H 3268 8173 50  0000 C CNN
-F 2 "" H 3250 8000 50  0001 C CNN
-F 3 "" H 3250 8000 50  0001 C CNN
-	1    3250 8000
-	0    1    1    0
-$EndComp
-$Comp
 L power:VDD #PWR011
 U 1 1 5DA1787C
@@
 	1    0    0    -1
 $EndComp
-Wire Wire Line
-	13650 2400 14150 2400
-Wire Wire Line
-	14150 2400 14150 2300
-Connection ~ 14150 2300
-$Comp
-L badge-rescue:Conn_01x04 J3
-U 1 1 5DA62B7B
-P 3000 7800
-F 0 "J3" H 2918 8117 50  0000 C CNN
-F 1 "AA Batteries " H 2918 8026 50  0000 C CNN
-F 2 "Dragos:AA" H 3000 7800 50  0001 C CNN
-F 3 "" H 3000 7800 50  0001 C CNN
-	1    3000 7800
-	-1   0    0    -1
-$EndComp
-$Comp
-L power:VDD #PWR0102
-U 1 1 5DA63097
-P 3250 7700
-F 0 "#PWR0102" H 3250 7550 50  0001 C CNN
-F 1 "VDD" H 3267 7873 50  0000 C CNN
-F 2 "" H 3250 7700 50  0001 C CNN
-F 3 "" H 3250 7700 50  0001 C CNN
-	1    3250 7700
-	0    1    1    0
-$EndComp
-Wire Wire Line
-	3200 7800 3250 7800
-Wire Wire Line
-	3250 7800 3250 7900
-Wire Wire Line
-	3250 7900 3200 7900
-Wire Wire Line
-	3200 8000 3250 8000
-Wire Wire Line
-	3200 7700 3250 7700
 $Comp
 L Device:LED_BGRA D1
@@
 	0    -1   -1   0
 $EndComp
+Text GLabel 6100 5700 0    50   Input ~ 0
+Up
+$Comp
+L power:+5V #PWR0102
+U 1 1 5DAA8DF2
+P 13800 2400
+F 0 "#PWR0102" H 13800 2250 50  0001 C CNN
+F 1 "+5V" V 13815 2528 50  0000 L CNN
+F 2 "" H 13800 2400 50  0001 C CNN
+F 3 "" H 13800 2400 50  0001 C CNN
+	1    13800 2400
+	0    1    1    0
+$EndComp
+Wire Wire Line
+	13650 2400 13800 2400
+$Comp
+L badge-rescue:Conn_01x02 J1
+U 1 1 5DAB1D17
+P 3850 7950
+F 0 "J1" H 3768 7625 50  0000 C CNN
+F 1 "Conn_01x02" H 3768 7716 50  0000 C CNN
+F 2 "" H 3850 7950 50  0001 C CNN
+F 3 "" H 3850 7950 50  0001 C CNN
+	1    3850 7950
+	-1   0    0    1
+$EndComp
+$Comp
+L power:VDD #PWR0105
+U 1 1 5DAB203E
+P 4100 7850
+F 0 "#PWR0105" H 4100 7700 50  0001 C CNN
+F 1 "VDD" H 4117 8023 50  0000 C CNN
+F 2 "" H 4100 7850 50  0001 C CNN
+F 3 "" H 4100 7850 50  0001 C CNN
+	1    4100 7850
+	0    1    1    0
+$EndComp
+$Comp
+L power:VSS #PWR0106
+U 1 1 5DAB2353
+P 4100 8000
+F 0 "#PWR0106" H 4100 7850 50  0001 C CNN
+F 1 "VSS" H 4118 8173 50  0000 C CNN
+F 2 "" H 4100 8000 50  0001 C CNN
+F 3 "" H 4100 8000 50  0001 C CNN
+	1    4100 8000
+	0    1    1    0
+$EndComp
+Wire Wire Line
+	4050 7850 4100 7850
+Wire Wire Line
+	4050 7950 4100 7950
+Wire Wire Line
+	4100 7950 4100 8000
 $EndSCHEMATC

Commit message: Added ATGM336H test board
Parts:
- J1: symbol badge-rescue:Conn_01x02 -> dragos-rescue:Conn_01x02-badge-rescue
- J2: symbol badge-rescue:Conn_01x04 -> dragos-rescue:Conn_01x04-badge-rescue
Changed lines of the file:
@@
 EESchema Schematic File Version 4
-LIBS:power
-LIBS:74xx
-LIBS:dragos-cache
 EELAYER 30 0
 EELAYER END
@@
 	5900 4150 6000 4150
 $Comp
-L badge-rescue:Conn_01x04 J2
+L dragos-rescue:Conn_01x04-badge-rescue J2
 U 1 1 5DA2C918
 P 8600 6450
@@
 	13650 2400 13800 2400
 $Comp
-L badge-rescue:Conn_01x02 J1
+L dragos-rescue:Conn_01x02-badge-rescue J1
 U 1 1 5DAB1D17
 P 3850 7950
