File: Tests/ATGM336H/Schematics/ATGM336H.kicad_pcb (KiCad board)
At the start: 2 copper layers, 51.5 x 22.2 mm, 20 parts, among them J1 USB_C_Receptacle, J2 Conn_01x05, J3 Conn_01x05, J4 Cuttable Trace, J5 Cuttable Trace, J6 Conn_01x01, J7 Conn_01x01, U1 otter_CH330, U2 TLV1117-33, U4 ATGM336H-5N

Commit message: Finished FJE badge:
Parts:
- added Ref**: Val**, NFCBuisness:W, F.Cu at (116.8, 72.5)
- added Ref**: Val**, ATGM336H:GPSLogo, F.Cu at (130.5, 63.2)
- <- On: renamed from Power->1
Routing:
- net D-: track 10.00 -> 14.5 mm, vias 0 -> 2
- net D+: track 9.68 -> 12.8 mm
- net Net-(J1-PadB5): track 10.8 -> 11.6 mm
- net Net-(J1-PadA5): track 9.27 -> 9.78 mm
Other:
- board text added: "@RMA_Electronics"
- board text added: "Cut J4 and J5 to disconnect USB UART"
- board text added: "Open Pins"
- board text added: "V1"
