File: Badges/FireJumperElite/Schematics/FJE Badge.kicad_pcb (KiCad board)
At the start: 2 copper layers, 88.7 x 89.8 mm, 45 parts, among them J1 USB_C_Receptacle, J2 Prog, J3 Conn_02x03_Odd_Even, J4 Conn_02x03_Odd_Even, SW1 SW_DIP_x01, SW2 SW_DIP_x01, SW3 SW_DIP_x01, U1 TLV1117-33, U2 HX4056, U3 STM32F042F6Px

Commit message: Progress on FJE firmware
Parts:
- removed the G*** at (155.2, 96.5) (x3)
- added G*** (x3): LOGO, LOGO, F.Cu at (155.2, 96.5)
Changed lines of the file:
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@@
   (page A4)
   (layers
-    (0 F.Cu signal)
+    (0 F.Cu signal hide)
     (31 B.Cu signal)
     (32 B.Adhes user)
     (33 F.Adhes user)
-    (34 B.Paste user)
-    (35 F.Paste user)
-    (36 B.SilkS user)
-    (37 F.SilkS user)
+    (34 B.Paste user hide)
+    (35 F.Paste user hide)
+    (36 B.SilkS user hide)
+    (37 F.SilkS user hide)
     (38 B.Mask user)
     (39 F.Mask user hide)
