File: Badges/BlueTeamCon/Schematics/BlueTeamCon.sch (KiCad schematic (older format))
At the start: 72 parts, among them CN1 100nF, J1 USB_C_Receptacle, J2 Prog, J3 Conn_02x03_Odd_Even, J4 Conn_02x03_Odd_Even, SW1 SW_DIP_x01, U1 STM32F072CBTx, U3 HX4056, U4 TLV1117-33

Commit message: Further
Parts:
- BT1: footprint Battery:BatteryHolder_Keystone_3008_1x2450 -> Tests:Dongguan14500
- D10, D11, D12, D14, D15, D16, D17, D18, D2, D20, D21, D22, D23, D24, D25, D26, D27, D28, D29, D3, D30, D31, D32, D33, D34, D35, D36, D37, D38, D4, D5, D6, D8, D9: footprint (none) -> LED_SMD:LED_0805_2012Metric
- D39, D40, D41, D42: footprint (none) -> Dragos:T776-ReverseMountLED
- R1: footprint (none) -> Resistors_SMD:R_0805
- RN2, RN3, RN4: footprint (none) -> Resistors_SMD:R_Array_Convex_4x0603
- gave numbers to parts that had none: 3
Connections:
- net Int1: now also U2.11 (INT1)
- net Int2: now also U2.9 (INT2)
- no-connect marks 38 -> 41

Commit message: Updates
Parts:
- added R4: R_Small, Resistor_SMD:R_0805_2012Metric, symbol Device:R_Small
- added RN5: R_Pack04, Resistor_SMD:R_Array_Convex_4x0603, symbol Device:R_Pack04
- BT1: footprint Tests:Dongguan14500 -> Battery:BatteryHolder_Keystone_3008_1x2450
- R1: footprint Resistors_SMD:R_0805 -> Resistor_SMD:R_0805_2012Metric
- RN2, RN3, RN4: footprint Resistors_SMD:R_Array_Convex_4x0603 -> Resistor_SMD:R_Array_Convex_4x0603
Connections:
- net C1: now also D10.1 (K), D18.1 (K), D22.1 (K), D24.1 (K), D29.1 (K), D33.1 (K), D36.1 (K), D38.1 (K), U1.10 (PA0); no longer D13.1 (K), D19.1 (K), D25.1 (K), D31.1 (K), D37.1 (K), D7.1 (K), U1.46 (PB9)
- net C2: now also D11.1 (K), D19.1 (K), D25.1 (K), D30.1 (K), D34.1 (K), D37.1 (K), U1.4 (PC15); no longer D14.1 (K), D20.1 (K), D26.1 (K), D32.1 (K), D38.1 (K), D8.1 (K), U1.21 (PB10)
- net C3: now also D12.1 (K), D26.1 (K), D31.1 (K), D35.1 (K), U1.3 (PC14); no longer D15.1 (K), D21.1 (K), D27.1 (K), D33.1 (K), D9.1 (K), U1.22 (PB11)
- net C4: now also D13.1 (K), D27.1 (K), D32.1 (K), U1.2 (PC13); no longer D10.1 (K), D16.1 (K), D22.1 (K), D28.1 (K), D34.1 (K), U1.25 (PB12)
- net C5: now also D14.1 (K), D28.1 (K), U1.46 (PB9); no longer D11.1 (K), D17.1 (K), D23.1 (K), D29.1 (K), D35.1 (K), U1.26 (PB13)
- net C6: now also D15.1 (K), D20.1 (K), D23.1 (K), U1.45 (PB8); no longer D12.1 (K), D18.1 (K), D24.1 (K), D30.1 (K), D36.1 (K), U1.27 (PB14)
- net Hour: now also U1.30 (PA9); no longer U1.15 (PA5)
- net Int1: now also U1.27 (PB14); no longer U1.17 (PA7)
- net Int2: now also U1.26 (PB13); no longer U1.16 (PA6)
- net R1: now also U1.19 (PB1); no longer U1.18 (PB0)
- net R2: now also U1.18 (PB0); no longer U1.19 (PB1)
- net R3: now also U1.17 (PA7); no longer U1.20 (PB2)
- net R4: now also U1.16 (PA6); no longer U1.39 (PB3)
- net R5: now also U1.15 (PA5); no longer U1.40 (PB4)
- net R6: now also U1.14 (PA4); no longer U1.41 (PB5)
- net R7: now also U1.13 (PA3); no longer U1.45 (PB8)
- net S1: now also U1.25 (PB12); no longer U1.10 (PA0)
- net S2: now also U1.22 (PB11); no longer U1.11 (PA1)
- net S3: now also U1.21 (PB10); no longer U1.12 (PA2)
- net S4: now also U1.20 (PB2); no longer U1.13 (PA3)
- net SCL: now also RN5.2 (R2.1)
- net SDA: now also RN5.1 (R1.1)
- net VCC: now also RN5.5 (R4.2), RN5.6 (R3.2), RN5.7 (R2.2), RN5.8 (R1.2)
- net at D1.2 (A), D2.2 (A), D3.2 (A)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: now also D7.2 (A), D8.2 (A), D9.2 (A)
- net at D10.2 (A), D11.2 (A), D12.2 (A)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: now also D13.2 (A), D14.2 (A), D15.2 (A), D16.2 (A), D17.2 (A); no longer D7.2 (A), D8.2 (A), D9.2 (A)
- net at D25.2 (A), D26.2 (A), D27.2 (A)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: now also D24.2 (A); no longer D29.2 (A), D30.2 (A)
- net R8: now reaches RN3.4 (R4.1)
- net R8: now also U1.12 (PA2)
- net at RN3.5 (R4.2): now also D36.2 (A), D37.2 (A)
- net at RN4.5 (R4.2): now also D39.2 (A); no longer D42.2 (A)
- net at RN4.6 (R3.2): now also D40.2 (A); no longer D41.2 (A)
- net at RN4.7 (R2.2): now also D41.2 (A); no longer D40.2 (A)
- net at RN4.8 (R1.2): now also D42.2 (A); no longer D39.2 (A)
- new net: D18.2 (A), D19.2 (A), D20.2 (A), D21.2 (A), RN2.6 (R3.2)
- new net: D22.2 (A), D23.2 (A), RN2.5 (R4.2)
- new net: D29.2 (A), D30.2 (A), D31.2 (A), D32.2 (A), RN3.7 (R2.2)
- new net: D33.2 (A), D34.2 (A), D35.2 (A), RN3.6 (R3.2)
- new net: D38.2 (A), R4.1
- new net C7: D16.1 (K), D21.1 (K), D7.1 (K), U1.41 (PB5)
- new net C8: D17.1 (K), D8.1 (K), U1.40 (PB4)
- new net C9: D9.1 (K), U1.39 (PB3)
- new net R9: R4.2, U1.11 (PA1)
- no-connect marks 41 -> 36
Other:
- note added: "ADC Input"
- moved on the sheet: C6, C7, D10, D11, D12, D13, D14, D15, D16, D17, D18, D19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
