File: Badges/BlueTeamCon/Schematics/BlueTeamCon.kicad_pcb (KiCad board)
At the start: 2 copper layers, 104.9 x 91.1 mm, 79 parts, among them CN1 100nF, J1 USB_C_Receptacle, J2 Prog, SW1 SW_DIP_x01, U1 STM32F072CBTx, U2 LIS3DH, U3 HX4056, U4 TLV1117-33

Commit message: Updated schematic for new chip
Parts:
- removed C1, C2: 4.7uF, Capacitor_SMD:C_0805_2012Metric
- removed C3: 1uF, Capacitor_SMD:C_0805_2012Metric
- removed C4: 10nF, Capacitor_SMD:C_0805_2012Metric
- removed the G*** at (142.7, 100.8) (x3)
- removed J2: Prog, Connector_PinHeader_2.54mm:PinHeader_1x05_P2.54mm_Vertical
- removed U1: STM32F072CBTx, Package_QFP:LQFP-48_7x7mm_P0.5mm
- added G*** (x3): LOGO, LOGO, F.Cu at (142.7, 100.8)
Routing:
- net VCC: track 215.1 -> 175.2 mm
- net SWCLK: track 13.9 -> 1.20 mm
- net +BATT: track 81.6 -> 75.3 mm, vias 5 -> 4
- net VSS: track 89.8 -> 85.5 mm, vias 30 -> 28
- net SCL: track 76.4 -> 73.2 mm, vias 2 -> 1
- net SDA: track 80.4 -> 77.3 mm, vias 2 -> 1
- net NRST: track 41.2 -> 39.7 mm, vias 2 -> 1
Other:
- net class Default removed
