File: Badges/BlueTeamCon/Schematics/BlueTeamCon.kicad_pcb (KiCad board)
At the start: 2 copper layers, 104.9 x 91.1 mm, 5 parts

Commit message: Further
Parts:
- removed the G*** at (0.00, 0.00) (x5)
- added BT1: Battery_Cell, Tests:Dongguan14500, B.Cu at (143.1, 86.2)
- added C1: 4.7uF, Capacitor_SMD:C_0805_2012Metric, B.Cu at (153.3, 109.6)
- added C10: 10uF, Capacitor_SMD:C_0805_2012Metric, B.Cu at (174.4, 124.1)
- added C11: 1uF, Capacitor_SMD:C_0805_2012Metric, B.Cu at (156.3, 100.4)
- added C12: 1uF, Capacitor_SMD:C_0805_2012Metric, B.Cu at (174.6, 119.3)
- added C2: 4.7uF, Capacitor_SMD:C_0805_2012Metric, B.Cu at (181.6, 104.5)
- added C3: 1uF, Capacitor_SMD:C_0805_2012Metric, B.Cu at (163.3, 102.5)
- added C4: 10nF, Capacitor_SMD:C_0805_2012Metric, B.Cu at (163.3, 99.3)
- added C5: 10nF, Capacitor_SMD:C_0805_2012Metric, B.Cu at (143.9, 95.1)
- added C6: 10uF, Capacitor_SMD:C_0805_2012Metric, B.Cu at (170.0, 124.1)
- added C7: 100nF, Capacitor_SMD:C_0805_2012Metric, B.Cu at (154.0, 95.6)
- added C9: 10uF, Capacitor_SMD:C_0805_2012Metric, B.Cu at (159.6, 109.0)
- added CN1: 100nF, Resistor_SMD:R_Array_Convex_4x0603, B.Cu at (177.0, 92.5)
- added D1: LED, LED_SMD:LED_0805_2012Metric, F.Cu at (115.5, 109.6)
- added D10: LED, LED_SMD:LED_0805_2012Metric, F.Cu at (118.1, 111.7)
- added D11: LED, LED_SMD:LED_0805_2012Metric, F.Cu at (125.0, 111.9)
- added D12: LED, LED_SMD:LED_0805_2012Metric, F.Cu at (131.9, 111.7)
- added D13: LED, LED_SMD:LED_0805_2012Metric, F.Cu at (139.1, 111.9)
- added D14: LED, LED_SMD:LED_0805_2012Metric, F.Cu at (146.2, 111.7)
- added D15: LED, LED_SMD:LED_0805_2012Metric, F.Cu at (153.2, 111.8)
- added D16: LED, LED_SMD:LED_0805_2012Metric, F.Cu at (160.2, 111.8)
- added D17: LED, LED_SMD:LED_0805_2012Metric, F.Cu at (167.2, 111.9)
- added D18: LED, LED_SMD:LED_0805_2012Metric, F.Cu at (121.4, 115.5)
- added D19: LED, LED_SMD:LED_0805_2012Metric, F.Cu at (128.2, 115.2)
- added D2: LED, LED_SMD:LED_0805_2012Metric, F.Cu at (122.0, 109.0)
- added D20: LED, LED_SMD:LED_0805_2012Metric, F.Cu at (156.9, 115.5)
- added D21: LED, LED_SMD:LED_0805_2012Metric, F.Cu at (163.6, 115.2)
- added D22: LED, LED_SMD:LED_0805_2012Metric, F.Cu at (125.1, 118.7)
- added D23: LED, LED_SMD:LED_0805_2012Metric, F.Cu at (160.2, 118.8)
- added D24: LED, LED_SMD:LED_0805_2012Metric, F.Cu at (128.6, 122.5)
- added D25: LED, LED_SMD:LED_0805_2012Metric, F.Cu at (136.0, 122.9)
- added D26: LED, LED_SMD:LED_0805_2012Metric, F.Cu at (143.2, 123.0)
- added D27: LED, LED_SMD:LED_0805_2012Metric, F.Cu at (150.2, 122.9)
- added D28: LED, LED_SMD:LED_0805_2012Metric, F.Cu at (156.7, 122.4)
- added D29: LED, LED_SMD:LED_0805_2012Metric, F.Cu at (132.2, 125.8)
- added D3: LED, LED_SMD:LED_0805_2012Metric, F.Cu at (128.8, 108.6)
- added D30: LED, LED_SMD:LED_0805_2012Metric, F.Cu at (139.0, 125.8)
- added D31: LED, LED_SMD:LED_0805_2012Metric, F.Cu at (146.2, 125.9)
- added D32: LED, LED_SMD:LED_0805_2012Metric, F.Cu at (153.2, 125.9)
- added D33: LED, LED_SMD:LED_0805_2012Metric, F.Cu at (135.5, 129.4)
- added D34: LED, LED_SMD:LED_0805_2012Metric, F.Cu at (142.5, 129.3)
- added D35: LED, LED_SMD:LED_0805_2012Metric, F.Cu at (149.4, 129.2)
- added D36: LED, LED_SMD:LED_0805_2012Metric, F.Cu at (139.2, 132.8)
- added D37: LED, LED_SMD:LED_0805_2012Metric, F.Cu at (146.2, 132.9)
- added D38: LED, LED_SMD:LED_0805_2012Metric, F.Cu at (142.3, 136.3)
- added D39: LED, Dragos:T776-ReverseMountLED, B.Cu at (119.3, 72.2)
- added D4: LED, LED_SMD:LED_0805_2012Metric, F.Cu at (135.9, 108.6)
- added D40: LED, Dragos:T776-ReverseMountLED, B.Cu at (134.6, 72.2)
- added D41: LED, Dragos:T776-ReverseMountLED, B.Cu at (150.1, 72.3)
- added D42: LED, Dragos:T776-ReverseMountLED, B.Cu at (165.2, 72.3)
- added D5: LED, LED_SMD:LED_0805_2012Metric, F.Cu at (142.7, 108.6)
- added D6: LED, LED_SMD:LED_0805_2012Metric, F.Cu at (149.9, 108.6)
- added D7: LED, LED_SMD:LED_0805_2012Metric, F.Cu at (156.9, 108.7)
- added D8: LED, LED_SMD:LED_0805_2012Metric, F.Cu at (164.3, 109.0)
- added D9: LED, LED_SMD:LED_0805_2012Metric, F.Cu at (170.4, 109.3)
- added G*** (x4): LOGO, LOGO, F.Cu at (142.7, 100.8)
- added G***: LOGO, LOGO, F.Cu at (0.00, 0.00)
- added J1: USB_C_Receptacle, Tests:USB_C_Receptical-Jing, B.Cu at (187.8, 101.5)
- added J2: Prog, Connector_PinHeader_2.54mm:PinHeader_1x05_P2.54mm_Vertical, B.Cu at (191.3, 111.5)
- added Power->1: SW3, BreadBoardPwr:SK-3296S_switch, B.Cu at (192.8, 86.7)
- added R1: R_Small, Resistors_SMD:R_0805, B.Cu at (135.6, 98.9)
- added R2: 1.5, Resistor_SMD:R_0805_2012Metric, B.Cu at (148.3, 95.1)
- added R3: 1k, Resistor_SMD:R_0805_2012Metric, B.Cu at (158.3, 114.8)
- added REF**: 1pin, Connectors:1pin, F.Cu at (142.2, 57.4)
- added RN1: 1k, Resistor_SMD:R_Array_Convex_4x0603, B.Cu at (183.4, 92.6)
- added RN2: R_Pack04, Resistors_SMD:R_Array_Convex_4x0603, B.Cu at (122.8, 101.7)
- added RN3: R_Pack04, Resistors_SMD:R_Array_Convex_4x0603, B.Cu at (122.8, 96.9)
- added RN4: R_Pack04, Resistors_SMD:R_Array_Convex_4x0603, B.Cu at (107.4, 79.8)
- added SW1: SW_DIP_x01, Button_Switch_SMD:SW_SPST_SKQG_WithStem, B.Cu at (143.3, 134.6)
- added U1: STM32F072CBTx, Package_QFP:LQFP-48_7x7mm_P0.5mm, B.Cu at (173.4, 101.4)
- added U2: LIS3DH, Package_LGA:LGA-16_3x3mm_P0.5mm_LayoutBorder3x5y, B.Cu at (131.3, 98.1)
- added U3: HX4056, Package_SO:HTSOP-8-1EP_3.9x4.9mm_P1.27mm_EP2.4x3.2mm, B.Cu at (142.0, 103.0)
- added U4: TLV1117-33, Package_TO_SOT_SMD:SOT-223-3_TabPin2, B.Cu at (131.7, 109.3)
Routing:
- net VCC: track 0.00 -> 40.0 mm, vias 0 -> 2
- net NRST: track 0.00 -> 29.8 mm, vias 0 -> 2
- net Net-(J1-PadB5): track 0.00 -> 23.5 mm
- net SWDIO: track 0.00 -> 15.4 mm
- net Net-(J1-PadA5): track 0.00 -> 14.2 mm
- net D-: track 0.00 -> 13.2 mm
- net SWCLK: track 0.00 -> 12.9 mm
- net D+: track 0.00 -> 11.9 mm
- net VSS: track 0.00 -> 7.22 mm
- net +5V: track 0.00 -> 0.50 mm
Other:
- board text added: "+ - Clk SW Rst"

Commit message: Updates
Parts:
- removed the G*** at (142.7, 100.8) (x4)
- added G*** (x4): LOGO, LOGO, F.Cu at (142.7, 100.8)
- added R4: R_Small, Resistor_SMD:R_0805_2012Metric, B.Cu at (154.1, 103.6)
- added RN5: R_Pack04, Resistor_SMD:R_Array_Convex_4x0603, B.Cu at (106.8, 91.3)
- added Ref**: Val**, NFCBuisness:W, B.Cu at (95.7, 108.2)
- moved C6 70.4 mm to (105.3, 96.0), turned to 270 degrees
- moved U4 55.8 mm to (180.3, 82.0), turned to 180 degrees
- moved RN4 50.3 mm to (157.6, 76.8)
- moved C7 45.3 mm to (108.7, 96.0), turned to 270 degrees
- moved C10 40.4 mm to (150.4, 91.5), turned to 180 degrees
- moved R3 32.4 mm to (132.7, 95.0), turned to 180 degrees
- moved C9 32.1 mm to (132.6, 91.5)
- moved C12 31.4 mm to (178.0, 88.0)
- moved C11 30.0 mm to (183.7, 88.0)
- moved RN3 24.9 mm to (146.8, 103.6), turned to 270 degrees
- moved C5 24.1 mm to (163.2, 109.5), turned to 180 degrees
- moved R1 23.8 mm to (158.4, 105.8), turned to 180 degrees
- moved R2 20.4 mm to (128.2, 91.5)
- moved U2 17.8 mm to (113.7, 95.8), turned to 270 degrees
- moved C1 10.7 mm to (163.4, 105.9)
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- renumbered Power->1 to <-Power
Connections:
- D10 pad 1: C4 -> C1
- D11 pad 1: C5 -> C2
- D12 pad 1: C6 -> C3
- D13 pad 1: C1 -> C4
- D13 pad 2: Net-(D13-Pad2) -> Net-(D10-Pad2)
- D14 pad 1: C2 -> C5
- D14 pad 2: Net-(D13-Pad2) -> Net-(D10-Pad2)
- D15 pad 1: C3 -> C6
- D15 pad 2: Net-(D13-Pad2) -> Net-(D10-Pad2)
- D16 pad 1: C4 -> C7
- D16 pad 2: Net-(D13-Pad2) -> Net-(D10-Pad2)
- D17 pad 1: C5 -> C8
- D17 pad 2: Net-(D13-Pad2) -> Net-(D10-Pad2)
- D18 pad 1: C6 -> C1
- D18 pad 2: Net-(D13-Pad2) -> Net-(D18-Pad2)
- D19 pad 1: C1 -> C2
- D19 pad 2: Net-(D19-Pad2) -> Net-(D18-Pad2)
- D20 pad 1: C2 -> C6
- D20 pad 2: Net-(D19-Pad2) -> Net-(D18-Pad2)
- D21 pad 1: C3 -> C7
- D21 pad 2: Net-(D19-Pad2) -> Net-(D18-Pad2)
- D22 pad 1: C4 -> C1
- D22 pad 2: Net-(D19-Pad2) -> Net-(D22-Pad2)
- D23 pad 1: C5 -> C6
- D23 pad 2: Net-(D19-Pad2) -> Net-(D22-Pad2)
- D24 pad 1: C6 -> C1
- D24 pad 2: Net-(D19-Pad2) -> Net-(D24-Pad2)
- D25 pad 1: C1 -> C2
- D25 pad 2: Net-(D25-Pad2) -> Net-(D24-Pad2)
- D26 pad 1: C2 -> C3
- D26 pad 2: Net-(D25-Pad2) -> Net-(D24-Pad2)
- D27 pad 1: C3 -> C4
- D27 pad 2: Net-(D25-Pad2) -> Net-(D24-Pad2)
- D28 pad 1: C4 -> C5
- D28 pad 2: Net-(D25-Pad2) -> Net-(D24-Pad2)
- D29 pad 1: C5 -> C1
- D29 pad 2: Net-(D25-Pad2) -> Net-(D29-Pad2)
- D30 pad 1: C6 -> C2
- D30 pad 2: Net-(D25-Pad2) -> Net-(D29-Pad2)
- D31 pad 1: C1 -> C3
- D31 pad 2: Net-(D31-Pad2) -> Net-(D29-Pad2)
- D32 pad 1: C2 -> C4
- D32 pad 2: Net-(D31-Pad2) -> Net-(D29-Pad2)
- D33 pad 1: C3 -> C1
- D33 pad 2: Net-(D31-Pad2) -> Net-(D33-Pad2)
- D34 pad 1: C4 -> C2
- D34 pad 2: Net-(D31-Pad2) -> Net-(D33-Pad2)
- D35 pad 1: C5 -> C3
- D35 pad 2: Net-(D31-Pad2) -> Net-(D33-Pad2)
- D36 pad 1: C6 -> C1
- D36 pad 2: Net-(D31-Pad2) -> Net-(D36-Pad2)
- D37 pad 1: C1 -> C2
- D37 pad 2: Net-(D37-Pad2) -> Net-(D36-Pad2)
- D38 pad 1: C2 -> C1
- D38 pad 2: Net-(D37-Pad2) -> Net-(D38-Pad2)
- D7 pad 1: C1 -> C7
- D7 pad 2: Net-(D10-Pad2) -> Net-(D1-Pad2)
- D8 pad 1: C2 -> C8
- D8 pad 2: Net-(D10-Pad2) -> Net-(D1-Pad2)
- D9 pad 1: C3 -> C9
- D9 pad 2: Net-(D10-Pad2) -> Net-(D1-Pad2)
- RN2 pad 5: Net-(D19-Pad2) -> Net-(D22-Pad2)
- RN2 pad 6: Net-(D13-Pad2) -> Net-(D18-Pad2)
- RN3 pad 4: Net-(RN3-Pad4) -> R8
- RN3 pad 5: Net-(RN3-Pad5) -> Net-(D36-Pad2)
- RN3 pad 6: Net-(D37-Pad2) -> Net-(D33-Pad2)
- RN3 pad 7: Net-(D31-Pad2) -> Net-(D29-Pad2)
- RN3 pad 8: Net-(D25-Pad2) -> Net-(D24-Pad2)
- RN4 pad 5: Net-(D42-Pad2) -> Net-(D39-Pad2)
- RN4 pad 6: Net-(D41-Pad2) -> Net-(D40-Pad2)
- RN4 pad 7: Net-(D40-Pad2) -> Net-(D41-Pad2)
- RN4 pad 8: Net-(D39-Pad2) -> Net-(D42-Pad2)
- U1 pad 10: S1 -> C1
- U1 pad 11: S2 -> R9
- U1 pad 12: S3 -> R8
- U1 pad 13: S4 -> R7
- U1 pad 14: Net-(U1-Pad14) -> R6
- U1 pad 15: Hour -> R5
- U1 pad 16: Int2 -> R4
- U1 pad 17: Int1 -> R3
- U1 pad 18: R1 -> R2
- U1 pad 19: R2 -> R1
- U1 pad 2: Net-(U1-Pad2) -> C4
- U1 pad 20: R3 -> S4
- U1 pad 21: C2 -> S3
- U1 pad 22: C3 -> S2
- U1 pad 25: C4 -> S1
- U1 pad 26: C5 -> Int2
- U1 pad 27: C6 -> Int1
- U1 pad 3: Net-(U1-Pad3) -> C3
- U1 pad 30: Net-(U1-Pad30) -> Hour
- U1 pad 39: R4 -> C9
- U1 pad 4: Net-(U1-Pad4) -> C2
- U1 pad 40: R5 -> C8
- U1 pad 41: R6 -> C7
- U1 pad 45: R7 -> C6
- U1 pad 46: C1 -> C5
Routing:
- net +5V: track 0.50 -> 193.5 mm, vias 0 -> 3
- net VCC: track 40.0 -> 215.1 mm, vias 2 -> 0
- net C2: track 0.00 -> 110.8 mm, vias 0 -> 8
- net C1: track 0.00 -> 108.0 mm, vias 0 -> 1
- net Int1: track 0.00 -> 92.7 mm, vias 0 -> 2
- net Net-(D18-Pad2): track 0.00 -> 90.8 mm, vias 0 -> 2
- net Int2: track 0.00 -> 87.2 mm, vias 0 -> 2
- net VSS: track 7.22 -> 89.8 mm, vias 0 -> 30
- net +BATT: track 0.00 -> 81.6 mm, vias 0 -> 5
- net SDA: track 0.00 -> 80.4 mm, vias 0 -> 2
- net C3: track 0.00 -> 78.4 mm, vias 0 -> 6
- net SCL: track 0.00 -> 76.4 mm, vias 0 -> 2
- net Net-(D22-Pad2): track 0.00 -> 73.8 mm, vias 0 -> 2
- net C4: track 0.00 -> 69.9 mm, vias 0 -> 5
- net Hour: track 0.00 -> 64.8 mm, vias 0 -> 2
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- added copper zone on B.Cu, net VSS
- added copper zone on F.Cu, net VSS
Other:
- board text added: "@RMA_Electronics"
- board text added: "Do not replace with AA Battery"
- board text added: "Rst SW Clk - +"
- board text added: "This is a 14500 Rechargable Battery"
- board text added: "This is not a AA battery"
- board text added: "V1"
- board text removed: "+ - Clk SW Rst"

Commit message: Some cleanup
Parts:
- removed CN1: 100nF, Resistor_SMD:R_Array_Convex_4x0603
- removed the G*** at (142.7, 100.8) (x3)
- added C13: 100nF, Capacitor_SMD:C_0805_2012Metric, B.Cu at (178.0, 93.5)
- added C14: 100nF, Capacitor_SMD:C_0805_2012Metric, B.Cu at (163.3, 102.6)
- added C15: 100nF, Capacitor_SMD:C_0805_2012Metric, B.Cu at (178.0, 90.5)
- added C8: 100nF, Capacitor_SMD:C_0805_2012Metric, B.Cu at (167.2, 105.9)
- added G*** (x3): LOGO, LOGO, F.Cu at (142.7, 100.8)
- R1: value R_Small -> 100k; footprint Resistors_SMD:R_0805 -> Resistor_SMD:R_0805_2012Metric
- R4: value R_Small -> 330
- RN2, RN3: value R_Pack04 -> 330; footprint Resistors_SMD:R_Array_Convex_4x0603 -> Resistor_SMD:R_Array_Convex_4x0603
- RN4: value R_Pack04 -> 1k; footprint Resistors_SMD:R_Array_Convex_4x0603 -> Resistor_SMD:R_Array_Convex_4x0603
- RN5: value R_Pack04 -> 5.1k
- moved C3 1.10 mm to (163.4, 100.0)
- moved C12 0.55 mm to (178.0, 87.5)
- moved C4 0.33 mm to (163.4, 97.5)
- moved BT1 0.29 mm to (141.9, 84.1)
- renumbered <-Power to Power->1
Connections:
- J1 pad A8: Net-(J1-PadA8) -> unconnected-(J1-PadA8)
- J1 pad B8: Net-(J1-PadB8) -> unconnected-(J1-PadB8)
- Power->1 pad 1: Net-(Power->1-Pad1) -> unconnected-(Power->1-Pad1)
- RN1 pad 3: Net-(RN1-Pad3) -> unconnected-(RN1-Pad3)
- RN1 pad 4: Net-(RN1-Pad4) -> unconnected-(RN1-Pad4)
- RN1 pad 5: Net-(RN1-Pad5) -> unconnected-(RN1-Pad5)
- RN1 pad 6: Net-(RN1-Pad6) -> unconnected-(RN1-Pad6)
- RN5 pad 3: Net-(RN5-Pad3) -> unconnected-(RN5-Pad3)
- RN5 pad 4: Net-(RN5-Pad4) -> unconnected-(RN5-Pad4)
- U1 pad 28: Net-(U1-Pad28) -> unconnected-(U1-Pad28)
- U1 pad 29: Net-(U1-Pad29) -> unconnected-(U1-Pad29)
- U1 pad 31: Net-(U1-Pad31) -> unconnected-(U1-Pad31)
- U1 pad 38: Net-(U1-Pad38) -> unconnected-(U1-Pad38)
- U1 pad 5: Net-(U1-Pad5) -> unconnected-(U1-Pad5)
- U1 pad 6: Net-(U1-Pad6) -> unconnected-(U1-Pad6)
- U2 pad 13: Net-(U2-Pad13) -> unconnected-(U2-Pad13)
- U2 pad 15: Net-(U2-Pad15) -> unconnected-(U2-Pad15)
- U2 pad 16: Net-(U2-Pad16) -> unconnected-(U2-Pad16)
- U2 pad 2: Net-(U2-Pad2) -> unconnected-(U2-Pad2)
- U2 pad 3: Net-(U2-Pad3) -> unconnected-(U2-Pad3)
- U3 pad 6: Net-(U3-Pad6) -> unconnected-(U3-Pad6)
- U3 pad 7: Net-(U3-Pad7) -> unconnected-(U3-Pad7)
Routing:
- net VSS: track 89.8 -> 84.6 mm, vias 30 -> 29
- net VCC: track 215.1 -> 211.4 mm
- net C1: track 108.0 -> 109.6 mm
- net R1: track 57.3 -> 58.2 mm
- net R2: track 55.5 -> 56.4 mm
- net R3: track 53.8 -> 54.5 mm
- net R4: track 52.0 -> 52.7 mm
- net R5: track 32.0 -> 32.7 mm
- net R6: track 30.3 -> 31.0 mm
- net R7: track 28.3 -> 29.0 mm
- net R8: track 26.3 -> 27.0 mm
- net R9: track 19.2 -> 19.9 mm
Other:
- net class Default removed
- board text added: "V2"
- board text removed: "V1"
