File: Badges/BlueTeamCon/Schematics/BlueTeamCon.kicad_pcb (KiCad board)
At the start: 2 copper layers, 104.9 x 91.1 mm, 89 parts, among them J1 USB_C_Receptacle, J2 Prog, SW1 SW_DIP_x01, U1 STM32F072CBTx, U2 LIS3DH, U3 HX4056, U4 TLV1117-33

Commit message: Blue Team Con V3
Parts:
- removed svg2mod (x7): G***, svg2mod
- added ?: , buzzardLabel, F.Cu at (198.6, 82.2)
- added ?: , buzzardLabel, B.Cu at (189.0, 87.2)
- added ?: , buzzardLabel, B.Cu at (92.4, 96.6)
- added ?: , buzzardLabel, B.Cu at (96.6, 110.4)
- added ?: , buzzardLabel, B.Cu at (142.4, 113.4)
- added ?: , buzzardLabel, B.Cu at (187.2, 83.4)
- added ?: , buzzardLabel, B.Cu at (95.4, 90.8)
- added J5: Conn_01x02, Connector_PinHeader_2.54mm:PinHeader_1x02_P2.54mm_Vertical, B.Cu at (184.7, 92.4)
- added R5: 0 Ohm, Resistor_SMD:R_0805_2012Metric, B.Cu at (141.3, 88.4)
- moved Ref** 6.74 mm to (102.4, 107.5)
- moved RN1 5.23 mm to (183.6, 97.8), turned to 180 degrees
- moved C14 0.20 mm to (163.3, 102.6)
- moved R2 0.06 mm to (128.1, 91.5), turned to 180 degrees
- turned C9 to 180 degrees
- renumbered Power->1 to Power1
Connections:
- C11 pad 2: Net-(C11-Pad2) -> +BATT
- C12 pad 2: VCC -> Net-(C12-Pad2)
- C9 pad 1: Net-(C9-Pad1) -> +5V
- C9 pad 2: +5V -> Net-(C9-Pad2)
- Power1 pad 1: unconnected-(Power->1-Pad1) -> VDDA
- Power1 pad 2: +BATT -> VCC
- Power1 pad 3: Net-(C11-Pad2) -> Net-(C12-Pad2)
- R2 pad 1: VSS -> Net-(C9-Pad2)
- R2 pad 2: Net-(C9-Pad1) -> VSS
- RN1 pad 1: Net-(J1-PadB5) -> unconnected-(RN1-Pad1)
- RN1 pad 2: Net-(J1-PadA5) -> unconnected-(RN1-Pad2)
- RN1 pad 3: unconnected-(RN1-Pad3) -> Net-(J1-PadB5)
- RN1 pad 4: unconnected-(RN1-Pad4) -> Net-(J1-PadA5)
- RN1 pad 5: unconnected-(RN1-Pad5) -> VSS
- RN1 pad 6: unconnected-(RN1-Pad6) -> VSS
- RN1 pad 7: VSS -> unconnected-(RN1-Pad7)
- RN1 pad 8: VSS -> unconnected-(RN1-Pad8)
- U4 pad 2: VCC -> Net-(C12-Pad2)
- U4 pad 3: Net-(C11-Pad2) -> +BATT
Routing:
- net Net-(C12-Pad2): track 0.00 -> 21.9 mm
- net VSS: track 84.6 -> 101.0 mm, vias 31 -> 33
- net Net-(C11-Pad2): track 11.6 -> 0.00 mm
- net Net-(D39-Pad2): track 54.0 -> 65.4 mm
- net Net-(J1-PadA5): track 14.2 -> 3.14 mm
- net Net-(D41-Pad2): track 17.1 -> 26.2 mm
- net Net-(D40-Pad2): track 30.7 -> 39.2 mm
- net VDDA: track 0.00 -> 7.91 mm
- net VCC: track 214.0 -> 221.4 mm, vias 0 -> 2
- net +BATT: track 81.6 -> 88.7 mm
- net Net-(J1-PadB5): track 23.5 -> 16.6 mm
- net +5V: track 193.5 -> 198.3 mm
- net Net-(C9-Pad2): track 0.00 -> 2.67 mm
- net Net-(C9-Pad1): track 2.56 -> 0.00 mm
- net Net-(D24-Pad2): track 48.5 -> 47.9 mm
Other:
- board text added: "+"
- board text added: "Mode"
- board text removed: "Do not replace with AA Battery"
- board text removed: "V2"
