File: Badges/BlueTeamCon/Schematics/BlueTeamCon.kicad_sch (KiCad schematic)
At the start: 74 parts, among them CN1 100nF, J1 USB_C_Receptacle, J2 Prog, J3 Conn_02x03_Odd_Even, J4 Conn_02x03_Odd_Even, SW1 SW_DIP_x01, U1 STM32F072CBTx, U2 LIS3DH, U3 HX4056, U4 TLV1117-33

Commit message: Some cleanup
Parts:
- removed CN1: 100nF, Resistor_SMD:R_Array_Convex_4x0603, symbol Device:R_Pack04
- added C13, C14, C15, C8: 100nF, Capacitor_SMD:C_0805_2012Metric, symbol Device:C_Small
- BT1: footprint Battery:BatteryHolder_Keystone_3008_1x2450 -> Tests:Dongguan14500
Connections:
- net VCC: now also C13.2, C14.2, C15.2, C8.2
- net VSS: now also C13.1, C14.1, C15.1, C8.1
Other:
- moved on the sheet: C1, C2, C3, C4
