File: Badges/BlueTeamCon/Schematics/BlueTeamCon.kicad_sch (KiCad schematic)
At the start: 77 parts, among them J1 USB_C_Receptacle, J2 Prog, J3 Conn_02x03_Odd_Even, J4 Conn_02x03_Odd_Even, SW1 SW_DIP_x01, U1 STM32F072CBTx, U2 LIS3DH, U3 HX4056, U4 TLV1117-33

Commit message: Blue Team Con V3
Parts:
- removed C9: 10uF, Capacitor_SMD:C_0805_2012Metric, symbol badge-rescue:C
- removed J3, J4: Conn_02x03_Odd_Even, Connector_PinSocket_2.54mm:PinSocket_2x03_P2.54mm_Vertical, symbol Connector_Generic:Conn_02x03_Odd_Even
- added C9: 10uF, Capacitor_SMD:C_0805_2012Metric, symbol Device:C_Small
- added J5: Conn_01x02, Connector_PinHeader_2.54mm:PinHeader_1x02_P2.54mm_Vertical, symbol Connector_Generic:Conn_01x02
- added R5: 0 Ohm, Resistor_SMD:R_0805_2012Metric, symbol Device:R_Small
- renumbered Power->1 to Power1
Connections:
- net +5V: now also C9.1, R5.1
- net +BATT: now also C11.2, U4.3 (VI), R5.2; no longer Power1.2 (B)
- net VCC: now also Power1.2 (B); no longer C12.2, U4.2 (VO)
- net VSS: now also R2.2, RN1.5 (R4.2), RN1.6 (R3.2), J5.2 (Pin_2); no longer R2.1, RN1.7 (R2.2), RN1.8 (R1.2)
- net at J1.A5 (CC1): now also RN1.4 (R4.1); no longer RN1.2 (R2.1)
- net at J1.B5 (CC2): now also RN1.3 (R3.1); no longer RN1.1 (R1.1)
- net VDDA: now reaches Power1.1 (A)
- net VDDA: now also J5.1 (Pin_1)
- new net: C9.2, R2.1
- new net: C12.2, Power1.3 (C), U4.2 (VO)
- no-connect marks 36 -> 27
Other:
- moved on the sheet: BT1, C10, C11, C12, Power1, R2, R3, RN1, U3, U4

Commit message: BlueTeamCon firmware in progress
Other:
- note added: "This was a mistake. I should have kept the matrix whole. This adds significantly more programming"
Changed lines of the file:
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@@
     (stroke (width 0) (type solid) (color 0 0 0 0))
+  )
+  (text "This was a mistake. I should have kept the matrix whole. \nThis adds significantly more programming"
+    (at 167.64 17.78 0)
+    (effects (font (size 1.27 1.27)) (justify right bottom))
   )
   (text "ADC Input" (at 198.12 147.32 90)
@@
   (symbol (lib_id "Device:R_Small") (at 205.74 66.04 270) (unit 1)
     (in_bom yes) (on_board yes)
-    (property "Reference" "R1" (id 0) (at 205.74 61.0616 90))
+    (property "Reference" "R1" (id 0) (at 201.93 63.6016 90))
     (property "Value" "100k" (id 1) (at 205.74 63.373 90))
     (property "Footprint" "Resistor_SMD:R_0805_2012Metric" (id 2) (at 205.74 66.04 0)
