File: SAO/Python/Schmatics/Python.kicad_pcb (KiCad board)
At the start: 2 copper layers, 30.9 x 30.9 mm, 5 parts

Commit message: Updates
Parts:
- removed the G*** at (128.3, 108.0) (x3)
- added G*** (x3): LOGO, LOGO, F.Cu at (128.3, 108.0)
Changed lines of the file:
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@@
   (page A4)
   (layers
-    (0 F.Cu signal hide)
+    (0 F.Cu signal)
     (31 B.Cu signal)
     (32 B.Adhes user)
@@
       (effects (font (size 1 1) (thickness 0.15)) (justify mirror))
     )
-    (fp_text value TestPoint_Pad_D3.0mm (at 0 -2.55) (layer B.Fab)
+    (fp_text value TestPoint_Pad_D3.0mm (at 0 -2.55) (layer B.Fab) hide
       (effects (font (size 1 1) (thickness 0.15)) (justify mirror))
     )
     (fp_circle (center 0 0) (end 0 -1.75) (layer B.SilkS) (width 0.12))
     (fp_circle (center 0 0) (end 2 0) (layer B.CrtYd) (width 0.05))
-    (fp_text user %R (at 0 2.4) (layer B.Fab)
+    (fp_text user %R (at 0 2.4) (layer B.Fab) hide
       (effects (font (size 1 1) (thickness 0.15)) (justify mirror))
     )
