File: SAO/Tux/Schematics/Tux.kicad_pcb (KiCad board)
At the start: 2 copper layers, 28.1 x 31.1 mm, 7 parts

Commit message: Updates
Parts:
- removed the G*** at (152.5, 97.0) (x3)
- added G*** (x3): LOGO, LOGO, F.Cu at (152.5, 97.0)
Changed lines of the file:
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@@
-(kicad_pcb (version 20171130) (host pcbnew 5.1.2)
+(kicad_pcb (version 20171130) (host pcbnew 5.1.5)
   (general
     (thickness 1.6)
@@
       (effects (font (size 1 1) (thickness 0.15)) (justify mirror))
     )
-    (fp_text value TestPoint_Pad_D3.0mm (at 0 -2.55) (layer B.Fab)
+    (fp_text value TestPoint_Pad_D3.0mm (at 0 -2.55) (layer B.Fab) hide
       (effects (font (size 1 1) (thickness 0.15)) (justify mirror))
     )
     (fp_circle (center 0 0) (end 0 -1.75) (layer B.SilkS) (width 0.12))
     (fp_circle (center 0 0) (end 2 0) (layer B.CrtYd) (width 0.05))
-    (fp_text user %R (at 0 2.4) (layer B.Fab)
+    (fp_text user %R (at 0 2.4) (layer B.Fab) hide
       (effects (font (size 1 1) (thickness 0.15)) (justify mirror))
     )
