File: Tests/ADV7123/Schematics/ADV7123.sch (KiCad schematic (older format))
At the start: 12 parts

Commit message: Started ADV7123 test board
Parts:
- removed U?: LM285D-1.2, Package_SO:SOIC-8_3.9x4.9mm_P1.27mm, symbol Reference_Voltage:LM285D-1.2
- added C?: 1uF, symbol Device:C_Small
- added R?: 1kOhm, symbol Device:R_Small
- added U?: LM4040DBZ-2.0, Package_TO_SOT_SMD:SOT-23, symbol Reference_Voltage:LM4040DBZ-2.0
Connections:
- net VCC: now also R?.1
- net VSS: now also C?.1, U?.2 (A)
- net BLANK: now reaches U?.11 (BLANK)
- net SYNC: now reaches U?.12 (SYNC)
- net CLK: now reaches U?.24 (CLK)
- net at U?.36 (VREF): now also C?.2, R?.2, U?.1 (K)
- net RESET: now reaches U?.37 (RSET)
- net PSAVE: now reaches U?.38 (PSAVE)
Changed lines of the file:
@@
 	5000 3000 5400 3000
 $Comp
-L Reference_Voltage:LM285D-1.2 U?
-U 1 1 5E809BF6
-P 5150 2300
-F 0 "U?" H 5150 2516 50  0000 C CNN
-F 1 "LM285D-1.2" H 5150 2425 50  0000 C CNN
-F 2 "Package_SO:SOIC-8_3.9x4.9mm_P1.27mm" H 5150 2100 50  0001 C CIN
-F 3 "http://www.onsemi.com/pub_link/Collateral/LM285-D.PDF" H 5150 2300 50  0001 C CIN
-	1    5150 2300
+L Reference_Voltage:LM4040DBZ-2.0 U?
+U 1 1 5E80BE56
+P 5250 2350
+F 0 "U?" H 5300 2550 50  0000 C CNN
+F 1 "LM4040DBZ-2.0" H 5250 2450 50  0000 C CNN
+F 2 "Package_TO_SOT_SMD:SOT-23" H 5250 2150 50  0001 C CIN
+F 3 "http://www.ti.com/lit/ds/symlink/lm4040-n.pdf" H 5250 2350 50  0001 C CIN
+	1    5250 2350
+	-1   0    0    1
+$EndComp
+Wire Wire Line
+	5000 2900 5100 2900
+Wire Wire Line
+	5100 2900 5100 2350
+Connection ~ 5100 2350
+Wire Wire Line
+	5100 2350 5100 2150
+$Comp
+L Device:R_Small R?
+U 1 1 5E810E10
+P 5100 1950
+F 0 "R?" H 4950 2000 50  0000 L CNN
+F 1 "1kOhm" H 4800 1900 50  0000 L CNN
+F 2 "" H 5100 1950 50  0001 C CNN
+F 3 "~" H 5100 1950 50  0001 C CNN
+	1    5100 1950
 	1    0    0    -1
 $EndComp
+$Comp
+L Device:C_Small C?
+U 1 1 5E811657
+P 5250 2150
+F 0 "C?" V 5021 2150 50  0000 C CNN
+F 1 "1uF" V 5112 2150 50  0000 C CNN
+F 2 "" H 5250 2150 50  0001 C CNN
+F 3 "~" H 5250 2150 50  0001 C CNN
+	1    5250 2150
+	0    1    1    0
+$EndComp
+Wire Wire Line
+	5400 2350 5400 2150
+$Comp
+L power:VSS #PWR?
+U 1 1 5E8144B6
+P 5400 2050
+F 0 "#PWR?" H 5400 1900 50  0001 C CNN
+F 1 "VSS" H 5417 2223 50  0000 C CNN
+F 2 "" H 5400 2050 50  0001 C CNN
+F 3 "" H 5400 2050 50  0001 C CNN
+	1    5400 2050
+	1    0    0    -1
+$EndComp
+Wire Wire Line
+	5350 2150 5400 2150
+Connection ~ 5400 2150
+Wire Wire Line
+	5400 2150 5400 2050
+Wire Wire Line
+	5150 2150 5100 2150
+Connection ~ 5100 2150
+Wire Wire Line
+	5100 2150 5100 2050
+$Comp
+L power:VCC #PWR?
+U 1 1 5E817E31
+P 5100 1750
+F 0 "#PWR?" H 5100 1600 50  0001 C CNN
+F 1 "VCC" H 5117 1923 50  0000 C CNN
+F 2 "" H 5100 1750 50  0001 C CNN
+F 3 "" H 5100 1750 50  0001 C CNN
+	1    5100 1750
+	1    0    0    -1
+$EndComp
+Wire Wire Line
+	5100 1850 5100 1750
+Text GLabel 3300 3900 0    50   Input ~ 0
+BLANK
+Text GLabel 3300 4000 0    50   Input ~ 0
+SYNC
+Text GLabel 4700 4300 3    50   Input ~ 0
+CLK
+Text GLabel 4600 2550 1    50   Input ~ 0
+PSAVE
+Text GLabel 4700 2550 1    50   Input ~ 0
+RESET
+Text GLabel 2050 2100 2    50   Input ~ 0
+PSAVE
+Text GLabel 2050 2200 2    50   Input ~ 0
+RESET
+Text GLabel 2050 2400 2    50   Input ~ 0
+BLANK
+Text GLabel 2050 2300 2    50   Input ~ 0
+SYNC
+Text GLabel 2050 2500 2    50   Input ~ 0
+CLK
 $EndSCHEMATC

Commit message: Updates
Parts:
- removed U?: LM4040DBZ-2.0, Package_TO_SOT_SMD:SOT-23, symbol Reference_Voltage:LM4040DBZ-2.0
- added D1: D_Schottky, Package_TO_SOT_SMD:SOT-23, symbol Device:D_Schottky
- added J2: Conn_01x05, Connector_PinHeader_2.54mm:PinHeader_1x05_P2.54mm_Vertical, symbol Connector_Generic:Conn_01x05
- added J3: Conn_01x04, Connector_PinHeader_2.54mm:PinHeader_1x04_P2.54mm_Vertical, symbol Connector_Generic:Conn_01x04
- added R5, R6: 47, Resistor_SMD:R_0805_2012Metric, symbol Device:R_Small
- C1, C2, C3, C4: renamed from C?; footprint (none) -> Capacitor_SMD:C_0805_2012Metric
- J1, J4, J5: renamed from J?; footprint (none) -> Connector_PinHeader_2.54mm:PinHeader_1x10_P2.54mm_Vertical
- R1, R2, R3, R4: renamed from R?; footprint (none) -> Resistor_SMD:R_0805_2012Metric
- U2: renamed from U?; footprint (none) -> ADV7123:VGA-002
- U3: renamed from U?; footprint (none) -> Package_QFP:LQFP-48_7x7mm_P0.5mm
Connections:
- net BLANK: now also J2.4 (Pin_4)
- net CLK: now also J2.5 (Pin_5)
- net PSAVE: now also J2.2 (Pin_2)
- net RESET: now also J2.1 (Pin_1)
- net SYNC: now also J2.3 (Pin_3)
- net VSS: now also D1.2 (A)
- net at C1.2, R1.2, U3.36 (VREF): now also D1.1 (K)
- net SDA: now reaches U2.12 (SDA)
- net SDA: now also J3.2 (Pin_2)
- net at U2.13 (HSync): now also R5.2
- net at U2.14 (VSync): now also R6.2
- net SCL: now reaches U2.15 (SCL)
- net SCL: now also J3.1 (Pin_1)
- new net HSync: J3.4 (Pin_4), R5.1
- new net VSync: J3.3 (Pin_3), R6.1
- no-connect marks 0 -> 6
