File: SAO/BernieMittens/BernieMittensMetal.kicad_pcb (KiCad board)
At the start: 2 copper layers, 28.9 x 62.2 mm, 6 parts

Commit message: BlueTeamCon firmware in progress
Parts:
- removed the G*** at (0.00, 0.00) (x6)
- added G*** (x6): LOGO, LOGO, F.Cu at (0.00, 0.00)
Other:
- net class Default removed
