File: SAO/BernieMittens/_autosave-BernieMittensNoChair.kicad_pcb (KiCad board)
At the start: 2 copper layers, 28.9 x 62.2 mm, 13 parts, among them J1 Conn_02x03_Odd_Even

Commit message: BlueTeamCon firmware in progress
Parts:
- removed the ? at (152.9, 82.1)
- added svg2mod: G***, svg2mod, B.Cu at (152.6, 82.5)
