File: Badges/BSidesIA2022/Schematics/Bottom/LayoutBottom.kicad_pcb (KiCad board)
At the start: 2 copper layers, 69.9 x 136.6 mm, 49 parts, among them J1 Program, J14 Neopixel Expansion, J2 Left_IN, J3 Right_Out, J5 Conn_01x10, J6 Conn_01x01, J8 Conn_01x01, J9 Conn_01x01, P1 USB_C_Plug_corrected, SW1 SW_SPDT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

Commit message: Mostly final Corncon
Parts:
- added J11: Cap Sense, Bsides22:CapSense, B.Cu at (132.6, 86.0)
- added J12: Cap Sense, Bsides22:CapSense, F.Cu at (110.2, 99.1)
- added J13: Cap Sense, Bsides22:CapSense, F.Cu at (172.2, 99.1)
- added Ref**: Val**, cafebabe:UELogoAbove, B.Cu at (158.0, 79.4)
- added Ref**: Val**, Bsides22:BackLogo, B.Cu at (181.1, 54.1)
- added kibuzzard-623F47EC: G***, kibuzzard-623F47EC, B.Cu at (163.4, 117.0)
- added kibuzzard-623F48F6: G***, kibuzzard-623F48F6, B.Cu at (116.3, 120.6)
- added kibuzzard-623F4981: G***, kibuzzard-623F4981, B.Cu at (168.1, 105.1)
- added kibuzzard-623F49DD: G***, kibuzzard-623F49DD, B.Cu at (141.2, 92.8)
- added kibuzzard-623F4E8E: G***, kibuzzard-623F4E8E, B.Cu at (164.0, 133.2)
- J5: value Conn_01x10 -> Conn_01x06; footprint Connector_PinHeader_2.54mm:PinHeader_1x10_P2.54mm_Vertical -> Connector_PinHeader_2.54mm:PinHeader_1x06_P2.54mm_Vertical
- moved BZ1 1.64 mm to (167.0, 97.8)
- moved SW2 0.90 mm to (157.6, 104.8)
- moved J14 0.73 mm to (168.2, 109.2)
- moved U1 0.45 mm to (113.2, 108.2)
- moved R1 0.40 mm to (113.0, 100.6)
- moved C18 0.15 mm to (119.0, 109.5)
- moved BT2 0.10 mm to (141.0, 141.5), turned to 0 degrees
Connections:
- C15 pad 2: unconnected-(C15-Pad2) -> VSS
- J5 pad 4: 4 -> 6
- J5 pad 5: 5 -> 7
- J5 pad 6: 6 -> 8
- J8 pad 1: unconnected-(J8-Pin_1) -> Net-(J13-Pin_1)
- J9 pad 1: unconnected-(J9-Pin_1) -> Net-(J12-Pin_1)
- U3 pad 5: Net-(U3-GPIO5/TOUCH5/ADC1_CH4) -> Net-(J12-Pin_1)
- U3 pad 6: Net-(U3-GPIO6/TOUCH6/ADC1_CH5) -> Net-(J13-Pin_1)
Routing:
- net VBUS: track 0.00 -> 91.4 mm, vias 0 -> 3
- net Net-(J13-Pin_1): track 0.00 -> 42.1 mm, vias 0 -> 3
- net Net-(J12-Pin_1): track 0.00 -> 28.9 mm, vias 0 -> 2
- net VDDA: track 184.7 -> 208.0 mm
- net Net-(J11-Pin_1): track 0.00 -> 20.8 mm, vias 0 -> 1
- net VSS: track 26.9 -> 45.7 mm, vias 16 -> 47
- net /SK6812: track 0.00 -> 11.9 mm, vias 0 -> 2
- net Net-(U1-PROG): track 0.00 -> 9.92 mm, vias 0 -> 2
- net VCC: track 195.1 -> 204.7 mm
- net Extra: track 46.3 -> 38.8 mm
- net TopRight: track 44.3 -> 51.3 mm
- net Net-(U3-GPIO18/U1RXD/ADC2_CH7/DAC_2/CLK_OUT3): track 0.00 -> 6.89 mm, vias 0 -> 2
- net Net-(U5-Dout): track 35.6 -> 40.5 mm
- net Net-(D1-K): track 0.00 -> 4.26 mm
- net Net-(U2-Dout): track 22.7 -> 27.0 mm
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Other:
- board text added: "JLCJLCJLCJLC"
