File: Tests/ThingAAskAskedFor/Schematics/ThingAAskAskedFor.kicad_sch (KiCad schematic)
At the start: 10 parts

Commit message: Updating for picoducky
Parts:
- removed U: (no value), symbol Switch:SW_SPDT
- added J: Conn_01x06, symbol Connector_Generic:Conn_01x06
Connections:
- net 1: now also J.6 (Pin_6)
- net 2: now also J.5 (Pin_5)
- net Button1: now also U.6 (GPIO4); no longer U.4 (GPIO2)
- net Button2: now also U.7 (GPIO5); no longer U.5 (GPIO3)
- net Buzzer: now also U.10 (GPIO7); no longer U.7 (GPIO5)
- net SK6812: now also U.9 (GPIO6); no longer U.6 (GPIO4)
- net VSS: now also U.13 (GND), U.18 (GND), U.23 (GND), U.28 (GND), U.3 (GND), U.33 (AGND), U.38 (GND), U.42 (GND), U.8 (GND), J.3 (Pin_3), J.4 (Pin_4)
- net Cout: no longer names the net of U.6 (Pin_6)
- new net 3: J.2 (Pin_2), U.4 (GPIO2)
- new net 4: J.1 (Pin_1), U.5 (GPIO3)
- no-connect marks 0 -> 24
Other:
- moved on the sheet: U

Commit message: Update for hondouras trip
Parts:
- removed U (x2): (no value), symbol LED:SK6812
- removed U (x2): (no value), symbol Device:C_Small
- added C: C_Small, symbol Device:C_Small
- added D: SK6812, LED_SMD:LED_SK6812_PLCC4_5.0x5.0mm_P3.2mm, symbol LED:SK6812
- added D (x2): 1N4148W, Diode_SMD:D_SOD-123, symbol Diode:1N4148W
- added D (x2): LED_Small, symbol Device:LED_Small
- added J: Conn_01x03, symbol Connector_Generic:Conn_01x03
- added RN: R_Pack04, symbol Device:R_Pack04
- added SW (x2): SW_SPDT, symbol Switch:SW_SPDT
- added U: (no value), symbol PlasticFrog-rescue:USB_A-Connector
Connections:
- net SK6812: now also D.2 (DIN)
- net VCC: now also U.36 (3V3), C.2, D.3 (VDD); no longer U.2 (Pin_2)
- net VSS: now also C.1, D.1 (K), D.1 (K), D.1 (VSS), SW.2 (B), SW.2 (B)
- net eyes: now reaches U.11 (GPIO8)
- net eyes: now also D.2 (A)
- net Switch1A: now reaches U.12 (GPIO9)
- net Switch1A: now also SW.1 (A)
- net Switch1B: now reaches U.14 (GPIO10)
- net Switch1B: now also SW.3 (C)
- net Switch2A: now reaches U.15 (GPIO11)
- net Switch2A: now also SW.1 (A)
- net Switch2B: now reaches U.16 (GPIO12)
- net Switch2B: now also SW.3 (C)
- net VBUS: now reaches U.40 (VBUS)
- net VBUS: now also U.1 (VBUS)
- new net: D.1 (K), D.1 (K), RN.3 (R3.1), RN.4 (R4.1)
- new net: D.2 (A), RN.5 (R4.2)
- new net: D.2 (A), RN.6 (R3.2)
- new net: J.2 (Pin_2), U.2 (D-)
- new net: J.1 (Pin_1), U.3 (D+)
- new net: J.3 (Pin_3), U.4 (GND), U.5 (Shield)
- new net +3V3: D.2 (A), U.2 (Pin_2)
- no-connect marks 24 -> 28
Other:
- moved on the sheet: J, U
